File: Lines.kicad_pcb (KiCad board)
At the start: 2 copper layers, 29.5 x 106.5 mm, 79 parts, among them J1 AudioJack2_SwitchT, J10 AudioJack2_SwitchT, J11 AudioJack2_SwitchT, J12 AudioJack2_SwitchT, J13 AudioJack2_SwitchT, J14 AudioJack2_SwitchT, J15 AudioJack2_SwitchT, J16 AudioJack2_SwitchT, J17 Conn_02x05_Odd_Even, J2 AudioJack2_SwitchT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

Commit message: Complete power routing.
Parts:
- moved C10 15.5 mm to (134.6, 131.4), turned to 180 degrees
- moved C9 15.2 mm to (119.4, 131.4), turned to 180 degrees
- moved R31 2.73 mm to (119.4, 134.2)
- moved C3 0.13 mm to (119.4, 95.0)
Routing:
- net -12V: track 90.4 -> 124.3 mm
- net +12V: track 90.5 -> 123.9 mm
Changed lines of the file:
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@@
     (thickness 1.6)
     (drawings 71)
-    (tracks 35)
+    (tracks 69)
     (zones 0)
     (modules 79)
@@
   )
   (setup
-    (last_trace_width 1.27)
+    (last_trace_width 0.381)
+    (user_trace_width 0.381)
+    (user_trace_width 0.508)
+    (user_trace_width 0.635)
+    (user_trace_width 0.635)
+    (user_trace_width 1.016)
     (user_trace_width 1.27)
     (trace_clearance 0.2)
@@
   )
   (module Resistor_SMD:R_0603_1608Metric (layer B.Cu)
-    (at 119.4435 131.5085 180)
+    (at 119.4435 134.239 180)
     (descr "Resistor SMD 0603 (1608 Metric), square (rectangular) end terminal, IPC_7351 nominal, (Body size source: http://www.tortai-tech.com/upload/download/2011102023233369053.pdf), generated with kicad-footprint-generator")
     (tags resistor)
@@
   )
   (module Capacitor_SMD:C_0603_1608Metric (layer B.Cu)
-    (at 119.38 134.239)
+    (at 134.62 131.445 180)
     (descr "Capacitor SMD 0603 (1608 Metric), square (rectangular) end terminal, IPC_7351 nominal, (Body size source: http://www.tortai-tech.com/upload/download/2011102023233369053.pdf), generated with kicad-footprint-generator")
     (tags capacitor)
@@
     (fp_line (start -0.8 0.4) (end 0.8 0.4) (layer B.Fab) (width 0.1))
     (fp_line (start -0.8 -0.4) (end -0.8 0.4) (layer B.Fab) (width 0.1))
-    (pad 2 smd roundrect (at 0.7875 0) (size 0.875 0.95) (layers B.Cu B.Paste B.Mask) (roundrect_rratio 0.25)
+    (pad 2 smd roundrect (at 0.7875 0 180) (size 0.875 0.95) (layers B.Cu B.Paste B.Mask) (roundrect_rratio 0.25)
       (net 14 -12V))
-    (pad 1 smd roundrect (at -0.7875 0) (size 0.875 0.95) (layers B.Cu B.Paste B.Mask) (roundrect_rratio 0.25))
+    (pad 1 smd roundrect (at -0.7875 0 180) (size 0.875 0.95) (layers B.Cu B.Paste B.Mask) (roundrect_rratio 0.25))
     (model ${KISYS3DMOD}/Capacitor_SMD.3dshapes/C_0603_1608Metric.wrl
       (at (xyz 0 0 0))
@@
   )
   (module Capacitor_SMD:C_0603_1608Metric (layer B.Cu)
-    (at 134.62 131.445)
+    (at 119.38 131.445 180)
     (descr "Capacitor SMD 0603 (1608 Metric), square (rectangular) end terminal, IPC_7351 nominal, (Body size source: http://www.tortai-tech.com/upload/download/2011102023233369053.pdf), generated with kicad-footprint-generator")
     (tags capacitor)
@@
     (fp_line (start -0.8 0.4) (end 0.8 0.4) (layer B.Fab) (width 0.1))
     (fp_line (start -0.8 -0.4) (end -0.8 0.4) (layer B.Fab) (width 0.1))
-    (pad 2 smd roundrect (at 0.7875 0) (size 0.875 0.95) (layers B.Cu B.Paste B.Mask) (roundrect_rratio 0.25))
-    (pad 1 smd roundrect (at -0.7875 0) (size 0.875 0.95) (layers B.Cu B.Paste B.Mask) (roundrect_rratio 0.25)
+    (pad 2 smd roundrect (at 0.7875 0 180) (size 0.875 0.95) (layers B.Cu B.Paste B.Mask) (roundrect_rratio 0.25))
+    (pad 1 smd roundrect (at -0.7875 0 180) (size 0.875 0.95) (layers B.Cu B.Paste B.Mask) (roundrect_rratio 0.25)
       (net 13 +12V))
     (model ${KISYS3DMOD}/Capacitor_SMD.3dshapes/C_0603_1608Metric.wrl
@@
   )
   (module Capacitor_SMD:C_0603_1608Metric (layer B.Cu)
-    (at 119.507 94.996 180)
+    (at 119.38 94.996 180)
     (descr "Capacitor SMD 0603 (1608 Metric), square (rectangular) end terminal, IPC_7351 nominal, (Body size source: http://www.tortai-tech.com/upload/download/2011102023233369053.pdf), generated with kicad-footprint-generator")
     (tags capacitor)
@@
   (segment (start 113.194994 74.597006) (end 113.194994 92.837) (width 1.27) (layer B.Cu) (net 13))
   (segment (start 113.194994 92.837) (end 113.194994 119.634) (width 1.27) (layer B.Cu) (net 13))
-  (segment (start 113.194994 119.634) (end 113.194994 153.915068) (width 1.27) (layer B.Cu) (net 13))
+  (segment (start 113.194994 119.634) (end 113.194994 129.756006) (width 1.27) (layer B.Cu) (net 13))
+  (segment (start 113.194994 129.756006) (end 113.194994 153.915068) (width 1.27) (layer B.Cu) (net 13))
+  (segment (start 113.956994 93.599) (end 113.194994 92.837) (width 0.635) (layer B.Cu) (net 13))
+  (segment (start 118.74576 93.599) (end 113.956994 93.599) (width 0.635) (layer B.Cu) (net 13))
+  (segment (start 119.681148 94.534388) (end 118.74576 93.599) (width 0.635) (layer B.Cu) (net 13))
+  (segment (start 120.1675 94.996) (end 119.705888 94.534388) (width 0.635) (layer B.Cu) (net 13))
+  (segment (start 119.705888 94.534388) (end 119.681148 94.534388) (width 0.635) (layer B.Cu) (net 13))
+  (segment (start 113.232988 129.794) (end 113.194994 129.756006) (width 0.635) (layer B.Cu) (net 13))
+  (segment (start 118.745 129.794) (end 113.232988 129.794) (width 0.635) (layer B.Cu) (net 13))
+  (segment (start 120.0405 131.445) (end 120.0405 131.0895) (width 0.635) (layer B.Cu) (net 13))
+  (segment (start 120.0405 131.0895) (end 118.745 129.794) (width 0.635) (layer B.Cu) (net 13))
+  (segment (start 121.0565 132.461) (end 120.0405 131.445) (width 0.381) (layer B.Cu) (net 13))
+  (segment (start 126.238 132.461) (end 121.0565 132.461) (width 0.381) (layer B.Cu) (net 13))
+  (segment (start 127 130.4) (end 127 131.699) (width 0.381) (layer B.Cu) (net 13))
+  (segment (start 127 131.699) (end 126.238 132.461) (width 0.381) (layer B.Cu) (net 13))
+  (segment (start 120.705 94.996) (end 120.1675 94.996) (width 0.381) (layer B.Cu) (net 13))
+  (segment (start 125.857 94.996) (end 120.705 94.996) (width 0.381) (layer B.Cu) (net 13))
+  (segment (start 127 92.3) (end 127 93.853) (width 0.381) (layer B.Cu) (net 13))
+  (segment (start 127 93.853) (end 125.857 94.996) (width 0.381) (layer B.Cu) (net 13))
   (segment (start 138.811 68.875) (end 137.074 70.612) (width 1.27) (layer B.Cu) (net 14))
   (segment (start 138.811 65.8115) (end 138.811 68.875) (width 1.27) (layer B.Cu) (net 14))
   (segment (start 137.074 70.612) (end 140.804946 74.342946) (width 1.27) (layer B.Cu) (net 14))
-  (segment (start 140.804946 74.342946) (end 140.804946 108.839) (width 1.27) (layer B.Cu) (net 14))
-  (segment (start 140.804946 108.839) (end 140.804946 135.636) (width 1.27) (layer B.Cu) (net 14))
   (segment (start 140.804946 135.636) (end 140.804946 153.915068) (width 1.27) (layer B.Cu) (net 14))
+  (segment (start 140.790382 130.45249) (end 140.804946 130.467054) (width 0.635) (layer B.Cu) (net 14))
+  (segment (start 134.82501 130.45249) (end 140.790382 130.45249) (width 0.635) (layer B.Cu) (net 14))
+  (segment (start 133.8325 131.445) (end 134.82501 130.45249) (width 0.635) (layer B.Cu) (net 14))
+  (segment (start 140.804946 108.839) (end 140.804946 130.467054) (width 1.27) (layer B.Cu) (net 14))
+  (segment (start 140.804946 130.467054) (end 140.804946 135.636) (width 1.27) (layer B.Cu) (net 14))
+  (segment (start 134.743446 93.510054) (end 140.804946 93.510054) (width 0.635) (layer B.Cu) (net 14))
+  (segment (start 133.8325 94.421) (end 134.743446 93.510054) (width 0.635) (layer B.Cu) (net 14))
+  (segment (start 133.8325 94.996) (end 133.8325 94.421) (width 0.635) (layer B.Cu) (net 14))
+  (segment (start 140.804946 74.342946) (end 140.804946 93.510054) (width 1.27) (layer B.Cu) (net 14))
+  (segment (start 140.804946 93.510054) (end 140.804946 108.839) (width 1.27) (layer B.Cu) (net 14))
+  (segment (start 133.295 131.445) (end 133.8325 131.445) (width 0.381) (layer B.Cu) (net 14))
+  (segment (start 130.302 131.445) (end 133.295 131.445) (width 0.381) (layer B.Cu) (net 14))
+  (segment (start 127 136.3) (end 127 134.747) (width 0.381) (layer B.Cu) (net 14))
+  (segment (start 127 134.747) (end 130.302 131.445) (width 0.381) (layer B.Cu) (net 14))
+  (segment (start 133.295 94.996) (end 133.8325 94.996) (width 0.381) (layer B.Cu) (net 14))
+  (segment (start 128.938 94.996) (end 133.295 94.996) (width 0.381) (layer B.Cu) (net 14))
+  (segment (start 127 98.2) (end 127 96.934) (width 0.381) (layer B.Cu) (net 14))
+  (segment (start 127 96.934) (end 128.938 94.996) (width 0.381) (layer B.Cu) (net 14))
   (segment (start 128.27 52.451) (end 125.73 52.451) (width 1.27) (layer B.Cu) (net 27))
   (segment (start 115.443 57.277) (end 115.443 58.292) (width 1.27) (layer B.Cu) (net 27))

Commit message: Completed routing.
Connections:
- C10 pad 1: (no net) -> GND
- C13 pad 2: (no net) -> GND
- C14 pad 1: (no net) -> GND
- C3 pad 2: (no net) -> GND
- C4 pad 1: (no net) -> GND
- C9 pad 2: (no net) -> GND
- D3 pad 2: (no net) -> GND
- J1 pad S: (no net) -> GND
- J1 pad TN: (no net) -> GND
- J10 pad S: (no net) -> GND
- J11 pad S: (no net) -> GND
- J12 pad S: (no net) -> GND
- J13 pad S: (no net) -> GND
- J14 pad S: (no net) -> GND
- J15 pad S: (no net) -> GND
- J16 pad S: (no net) -> GND
- J17 pad 3: (no net) -> GND
- J17 pad 4: (no net) -> GND
- J17 pad 5: (no net) -> GND
- J17 pad 6: (no net) -> GND
- J17 pad 7: (no net) -> GND
- J17 pad 8: (no net) -> GND
- J2 pad S: (no net) -> GND
- J2 pad TN: (no net) -> GND
- J3 pad S: (no net) -> GND
- J3 pad TN: (no net) -> GND
- J4 pad S: (no net) -> GND
- J4 pad TN: (no net) -> GND
- J5 pad S: (no net) -> GND
- J5 pad TN: (no net) -> GND
- J6 pad S: (no net) -> GND
- J6 pad TN: (no net) -> GND
- J7 pad S: (no net) -> GND
- J7 pad TN: (no net) -> GND
- J8 pad S: (no net) -> GND
- J8 pad TN: (no net) -> GND
- J9 pad S: (no net) -> GND
- R13 pad 2: (no net) -> GND
- R14 pad 2: (no net) -> GND
- R15 pad 1: (no net) -> GND
- R16 pad 1: (no net) -> GND
- R23 pad 2: (no net) -> GND
- R24 pad 2: (no net) -> GND
- R25 pad 1: (no net) -> GND
- R26 pad 1: (no net) -> GND
- R3 pad 2: (no net) -> GND
- R33 pad 2: (no net) -> GND
- R34 pad 2: (no net) -> GND
- R35 pad 1: (no net) -> GND
- R36 pad 1: (no net) -> GND
- R4 pad 2: (no net) -> GND
- R5 pad 1: (no net) -> GND
- R6 pad 1: (no net) -> GND
Routing:
- net GND: track 0.00 -> 44.3 mm, vias 0 -> 19
- net Net-(C1-Pad1): track 0.00 -> 41.0 mm
- net Net-(R1-Pad1): track 0.00 -> 39.1 mm, vias 0 -> 2
- net Net-(R11-Pad1): track 0.00 -> 33.4 mm, vias 0 -> 2
- net Net-(R21-Pad1): track 0.00 -> 30.6 mm, vias 0 -> 2
- net Net-(C7-Pad1): track 0.00 -> 27.7 mm
- net Net-(D3-Pad1): track 0.00 -> 26.7 mm, vias 0 -> 2
- net Net-(C5-Pad1): track 0.00 -> 26.4 mm, vias 0 -> 2
- net Net-(R32-Pad1): track 0.00 -> 23.0 mm
- net Net-(R31-Pad1): track 0.00 -> 22.4 mm, vias 0 -> 2
- net Net-(C12-Pad1): track 0.00 -> 22.2 mm
- net Net-(R12-Pad1): track 0.00 -> 21.6 mm
- net Net-(R22-Pad1): track 0.00 -> 20.8 mm, vias 0 -> 2
- net Net-(C6-Pad1): track 0.00 -> 17.5 mm, vias 0 -> 2
- net Net-(C2-Pad1): track 0.00 -> 16.5 mm
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- added copper zone on B.Cu, net GND
- added copper zone on F.Cu, net GND

Commit message: Verified on breadboard and corrected input divider value.
Parts:
- R13, R14, R23, R24, R3, R33, R34, R4: value 47k -> 22k
Changed lines of the file:
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@@
       (effects (font (size 1 1) (thickness 0.15)) (justify mirror))
     )
-    (fp_text value 47k (at 0 -1.43) (layer B.Fab)
+    (fp_text value 22k (at 0 -1.43) (layer B.Fab)
       (effects (font (size 1 1) (thickness 0.15)) (justify mirror))
     )
@@
       (effects (font (size 1 1) (thickness 0.15)) (justify mirror))
     )
-    (fp_text value 47k (at 0 -1.43) (layer B.Fab)
+    (fp_text value 22k (at 0 -1.43) (layer B.Fab)
       (effects (font (size 1 1) (thickness 0.15)) (justify mirror))
     )
@@
       (effects (font (size 1 1) (thickness 0.15)) (justify mirror))
     )
-    (fp_text value 47k (at 0 -1.43) (layer B.Fab)
+    (fp_text value 22k (at 0 -1.43) (layer B.Fab)
       (effects (font (size 1 1) (thickness 0.15)) (justify mirror))
     )
@@
       (effects (font (size 1 1) (thickness 0.15)) (justify mirror))
     )
-    (fp_text value 47k (at 0 -1.43) (layer B.Fab)
+    (fp_text value 22k (at 0 -1.43) (layer B.Fab)
       (effects (font (size 1 1) (thickness 0.15)) (justify mirror))
     )
@@
       (effects (font (size 1 1) (thickness 0.15)) (justify mirror))
     )
-    (fp_text value 47k (at 0 -1.43) (layer B.Fab)
+    (fp_text value 22k (at 0 -1.43) (layer B.Fab)
       (effects (font (size 1 1) (thickness 0.15)) (justify mirror))
     )
@@
       (effects (font (size 1 1) (thickness 0.15)) (justify mirror))
     )
-    (fp_text value 47k (at 0 -1.43) (layer B.Fab)
+    (fp_text value 22k (at 0 -1.43) (layer B.Fab)
       (effects (font (size 1 1) (thickness 0.15)) (justify mirror))
     )
@@
       (effects (font (size 1 1) (thickness 0.15)) (justify mirror))
     )
-    (fp_text value 47k (at 0 -1.43) (layer B.Fab)
+    (fp_text value 22k (at 0 -1.43) (layer B.Fab)
       (effects (font (size 1 1) (thickness 0.15)) (justify mirror))
     )
@@
       (effects (font (size 1 1) (thickness 0.15)) (justify mirror))
     )
-    (fp_text value 47k (at 0 -1.43) (layer B.Fab)
-      (effects (font (size 1 1) (thickness 0.15)) (justify mirror))
-    )
+    (fp_text value 22k (at 0 -1.43) (layer B.Fab)
+      (effects (font (size 1 1) (thickness 0.15)) (justify mirror))
+    )

Commit message: Silk-screens.
Other:
- board text added: "+12V"
- board text added: "-12V"

Commit message: Branding.
Other:
- board text added: "Lines"
- board text added: "Marangisto 2019"
- board text added: "Rev A"
Changed lines of the file:
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@@
   (general
     (thickness 1.6)
-    (drawings 74)
+    (drawings 77)
     (tracks 399)
     (zones 0)
@@
     )
   )
+  (gr_text "Rev A" (at 139.827 78.232 90) (layer B.SilkS)
+    (effects (font (size 1 1) (thickness 0.15)) (justify mirror))
+  )
+  (gr_text "Marangisto 2019" (at 139.827 146.177 90) (layer B.SilkS)
+    (effects (font (size 1 1) (thickness 0.15)) (justify mirror))
+  )
+  (gr_text Lines (at 115.316 141.986 90) (layer B.SilkS)
+    (effects (font (size 3 6) (thickness 0.25)) (justify mirror))
+  )
   (gr_text +12V (at 127.254 50.165) (layer B.SilkS)
